File: usb_rs232_v1/_autosave-usb_rs232_converter_v1.kicad_pcb (KiCad board)
At the start: 2 copper layers, 59 x 40 mm, 46 parts, among them CON1 USB-micro-B, IC1 MAX3243, IC2 FT232BL, J1 COM LEFT, J2 COM RIGHT, J3 FTDI, J4 UART

Commit message: Pcb v0.2
Parts:
- C11, C7: moved to B.Cu
- COM1, COM3: footprint SIL-8-SMD -> SIL-8
- moved C10 93.5 mm to (160.7, 87.8), turned to 270 degrees
- moved C8 91.3 mm to (153.0, 87.6), turned to 0 degrees
- moved C7 90.6 mm to (158.0, 87.6), turned to 0 degrees
- moved C11 87.5 mm to (150.1, 89.9), turned to 270 degrees
- moved C3 82.2 mm to (152.6, 135.2)
- moved C5 67.2 mm to (139.7, 144.1)
- moved L1 67.2 mm to (140.7, 154.7)
- moved R1 67.2 mm to (145.7, 153.1)
- moved C2 67.2 mm to (140.9, 149.3)
- moved C9 67.2 mm to (146.5, 141.7)
- moved R2 67.2 mm to (134.3, 147.1)
- moved R3 67.2 mm to (133.3, 149.3)
- moved C12 67.2 mm to (138.1, 149.5)
- moved R4 67.2 mm to (136.5, 151.9)
- moved C4 67.2 mm to (142.1, 143.9)
Routing:
- net /DSR COM: track 48.9 -> 83.0 mm
- net /Rin: RI: track 0.00 -> 29.5 mm
- net /Rin: DCD: track 22.5 -> 3.12 mm
- net /RI COM LEFT: track 0.00 -> 18.8 mm
- net /Tout: RST: track 18.7 -> 4.09 mm
- net /RxD COM LEFT: track 0.00 -> 14.1 mm
- net /TxD COM LEFT: track 0.00 -> 10.4 mm
- net /RST COM LEFT: track 0.00 -> 9.94 mm
- net /DTR COM LEFT: track 0.00 -> 8.95 mm
- net /DSR COM LEFT: track 0.00 -> 6.43 mm
- net /CTS COM LEFT: track 0.00 -> 6.27 mm
- net N-000008: track 0.00 -> 5.79 mm
- net /DCD COM LEFT: track 0.00 -> 4.05 mm
- net N-0000014: track 0.00 -> 3.83 mm
- net N-0000015: track 0.00 -> 3.69 mm
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