File: usb_rs232_v1/usb_rs232_converter_v1-append.kicad_pcb (KiCad board)
At the start: 2 copper layers, 156.2 x 147.5 mm, 108 parts, among them CON1 USB-MINI-B, CON2 USB-MICRO-B, IC1 MAX3243, J1 DB9, J2 DB9

Commit message: PCB v1.1 poligony
Parts:
- removed the CON1 at (131.0, 113.5) (x3)
- removed the CON1 at (133.0, 169.0) (x2)
- removed the CON1 at (227.2, 61.5) (x4)
- removed the CON1 at (131.5, 66.2) (x6)
- removed the CON1 at (227.8, 163.5)
- removed the CON1 at (228.2, 116.2) (x2)
- removed the CON2 at (146.2, 116.8) (x3)
- removed the CON2 at (148.2, 172.2) (x2)
- removed the CON2 at (242.5, 64.8) (x4)
- removed the CON2 at (146.8, 69.5) (x6)
- removed the CON2 at (243.0, 166.8)
- removed the CON2 at (243.5, 119.5) (x2)
- removed I1 (x18): FT232BL, TQFP32
- removed the IC1 at (138.0, 84.2) (x3)
- removed the IC1 at (140.0, 139.8) (x2)
- removed the IC1 at (234.2, 32.2) (x4)
- removed the IC1 at (138.5, 37.0) (x6)
- removed the IC1 at (234.8, 134.2)
- removed the IC1 at (235.2, 87.0) (x2)
- removed the J1 at (121.1, 97.4) (x3)
- removed the J1 at (123.1, 152.9) (x2)
- removed the J1 at (217.3, 45.4) (x4)
- removed the J1 at (121.6, 50.2) (x6)
- removed the J1 at (217.8, 147.4)
- removed the J1 at (218.3, 100.2) (x2)
- removed the J2 at (155.1, 97.4) (x3)
- removed the J2 at (157.1, 152.9) (x2)
- removed the J2 at (251.3, 45.4) (x4)
- removed the J2 at (155.6, 50.2) (x6)
- removed the J2 at (251.8, 147.4)
- removed the J2 at (252.3, 100.2) (x2)
- added C10 (x3): C, SM0603_Capa, B.Cu at (178.3, 35.2)
- added C10 (x2): C, SM0603_Capa, B.Cu at (76.3, 91.2)
- added C10: C, SM0603_Capa, B.Cu at (181.3, 93.2)
- added C10: C, SM0603_Capa, B.Cu at (79.3, 157.2)
- added C10: C, SM0603_Capa, B.Cu at (74.3, 35.7)
- added C11 (x3): C, SM0603_Capa, B.Cu at (167.6, 35.7)
- added C11 (x2): C, SM0603_Capa, B.Cu at (65.6, 91.7)
- added C11: C, SM0603_Capa, B.Cu at (170.6, 93.7)
- added C11: C, SM0603_Capa, B.Cu at (68.6, 157.7)
- added C11: C, SM0603_Capa, B.Cu at (63.6, 36.2)
- added C12 (x3): 33n, SM0805, B.Cu at (156.5, 36.6)
- added C12 (x2): 33n, SM0805, B.Cu at (54.5, 92.6)
- added C12: 33n, SM0805, B.Cu at (159.5, 94.6)
- added C12: 33n, SM0805, B.Cu at (57.5, 158.6)
- added C12: 33n, SM0805, B.Cu at (52.5, 37.1)
- added C2 (x3): 100n, SM0603_Capa, F.Cu at (157.5, 46.6)
- added C2 (x2): 100n, SM0603_Capa, F.Cu at (55.5, 102.6)
- added C2: 100n, SM0603_Capa, F.Cu at (160.5, 104.6)
- added C2: 100n, SM0603_Capa, F.Cu at (58.5, 168.6)
- added C2: 100n, SM0603_Capa, F.Cu at (53.5, 47.1)
- added C3 (x3): 10u, SM1206POL, F.Cu at (157.5, 44.2)
- added C3 (x2): 10u, SM1206POL, F.Cu at (55.5, 100.2)
- added C3: 10u, SM1206POL, F.Cu at (160.5, 102.2)
- added C3: 10u, SM1206POL, F.Cu at (58.5, 166.2)
- added C3: 10u, SM1206POL, F.Cu at (53.5, 44.7)
- added C4 (x3): 100n, SM1206, F.Cu at (170.1, 41.2)
- added C4 (x2): 100n, SM1206, F.Cu at (68.1, 97.2)
- added C4: 100n, SM1206, F.Cu at (173.1, 99.2)
- added C4: 100n, SM1206, F.Cu at (71.1, 163.2)
- added C4: 100n, SM1206, F.Cu at (66.1, 41.7)
- added C5 (x3): 10u, SM1206POL, F.Cu at (170.1, 38.6)
- added C5 (x2): 10u, SM1206POL, F.Cu at (68.1, 94.6)
- added C5: 10u, SM1206POL, F.Cu at (173.1, 96.6)
- added C5: 10u, SM1206POL, F.Cu at (71.1, 160.6)
- added C5: 10u, SM1206POL, F.Cu at (66.1, 39.1)
- added C7 (x3): C, SM0603_Capa, B.Cu at (175.1, 33.0)
- added C7 (x2): C, SM0603_Capa, B.Cu at (73.1, 89.0)
- added C7: C, SM0603_Capa, B.Cu at (178.1, 91.0)
- added C7: C, SM0603_Capa, B.Cu at (76.1, 154.9)
- added C7: C, SM0603_Capa, B.Cu at (71.1, 33.5)
- added C8 (x3): C, SM0603_Capa, B.Cu at (171.6, 33.0)
- added C8 (x2): C, SM0603_Capa, B.Cu at (69.6, 89.0)
- added C8: C, SM0603_Capa, B.Cu at (174.6, 91.0)
- added C8: C, SM0603_Capa, B.Cu at (72.6, 154.9)
- added C8: C, SM0603_Capa, B.Cu at (67.6, 33.5)
- added C9 (x3): 100n, SM0603_Capa, B.Cu at (160.5, 50.2)
- added C9 (x2): 100n, SM0603_Capa, B.Cu at (58.5, 106.2)
- added C9: 100n, SM0603_Capa, B.Cu at (163.5, 108.2)
- added C9: 100n, SM0603_Capa, B.Cu at (61.5, 172.2)
- added C9: 100n, SM0603_Capa, B.Cu at (56.5, 50.7)
- added CON1 (x3): USB-micro-B, usb-micro-B, B.Cu at (149.2, 69.0)
- added CON1 (x2): USB-micro-B, usb-micro-B, B.Cu at (47.2, 125.0)
- added CON1: USB-micro-B, usb-micro-B, B.Cu at (152.2, 127.0)
- added CON1: USB-micro-B, usb-micro-B, B.Cu at (50.2, 191.0)
- added CON1: USB-micro-B, usb-micro-B, B.Cu at (45.2, 69.5)
- added CON2 (x3): USB-mini-B, usb-mini-B-2, B.Cu at (167.5, 65.5)
- added CON2 (x2): USB-mini-B, usb-mini-B-2, B.Cu at (65.5, 121.5)
- added CON2: USB-mini-B, usb-mini-B-2, B.Cu at (170.5, 123.5)
- added CON2: USB-mini-B, usb-mini-B-2, B.Cu at (68.5, 187.5)
- added CON2: USB-mini-B, usb-mini-B-2, B.Cu at (63.5, 66.0)
- added D1 (x3): RED, LED-3MM-SMD, F.Cu at (166.5, 45.4)
- added D1 (x2): RED, LED-3MM-SMD, F.Cu at (64.5, 101.4)
- added D1: RED, LED-3MM-SMD, F.Cu at (169.5, 103.4)
- added D1: RED, LED-3MM-SMD, F.Cu at (67.5, 167.4)
- added D1: RED, LED-3MM-SMD, F.Cu at (62.5, 45.9)
- added D11 (x3): RED, LED-3MM-SMD, F.Cu at (188.0, 51.8)
- added D11 (x2): RED, LED-3MM-SMD, F.Cu at (86.0, 107.8)
- added D11: RED, LED-3MM-SMD, F.Cu at (191.0, 109.8)
- added D11: RED, LED-3MM-SMD, F.Cu at (89.0, 173.8)
- added D11: RED, LED-3MM-SMD, F.Cu at (84.0, 52.2)
- added D12 (x3): GREEN, LED-3MM-SMD, F.Cu at (188.0, 47.0)
- added D12 (x2): GREEN, LED-3MM-SMD, F.Cu at (86.0, 103.0)
- added D12: GREEN, LED-3MM-SMD, F.Cu at (191.0, 105.0)
- added D12: GREEN, LED-3MM-SMD, F.Cu at (89.0, 169.0)
- added D12: GREEN, LED-3MM-SMD, F.Cu at (84.0, 47.5)
- added D13 (x3): YELLOW, LED-3MM-SMD, F.Cu at (187.8, 61.2)
- added D13 (x2): YELLOW, LED-3MM-SMD, F.Cu at (85.8, 117.2)
- added D13: YELLOW, LED-3MM-SMD, F.Cu at (190.8, 119.2)
- added D13: YELLOW, LED-3MM-SMD, F.Cu at (88.8, 183.2)
- added D13: YELLOW, LED-3MM-SMD, F.Cu at (83.8, 61.8)
- added D14 (x3): YELLOW, LED-3MM-SMD, F.Cu at (188.0, 42.2)
- added D14 (x2): YELLOW, LED-3MM-SMD, F.Cu at (86.0, 98.2)
- added D14: YELLOW, LED-3MM-SMD, F.Cu at (191.0, 100.2)
- added D14: YELLOW, LED-3MM-SMD, F.Cu at (89.0, 164.2)
- added D14: YELLOW, LED-3MM-SMD, F.Cu at (84.0, 42.8)
- added D15 (x3): YELLOW, LED-3MM-SMD, F.Cu at (188.0, 56.5)
- added D15 (x2): YELLOW, LED-3MM-SMD, F.Cu at (86.0, 112.5)
- added D15: YELLOW, LED-3MM-SMD, F.Cu at (191.0, 114.5)
- added D15: YELLOW, LED-3MM-SMD, F.Cu at (89.0, 178.5)
- added D15: YELLOW, LED-3MM-SMD, F.Cu at (84.0, 57.0)
- added D16 (x3): YELLOW, LED-3MM-SMD, F.Cu at (188.0, 37.5)
- added D16 (x2): YELLOW, LED-3MM-SMD, F.Cu at (86.0, 93.5)
- added D16: YELLOW, LED-3MM-SMD, F.Cu at (191.0, 95.5)
- added D16: YELLOW, LED-3MM-SMD, F.Cu at (89.0, 159.5)
- added D16: YELLOW, LED-3MM-SMD, F.Cu at (84.0, 38.0)
- added D17 (x3): YELLOW, LED-3MM-SMD, F.Cu at (188.0, 32.8)
- added D17 (x2): YELLOW, LED-3MM-SMD, F.Cu at (86.0, 88.8)
- added D17: YELLOW, LED-3MM-SMD, F.Cu at (191.0, 90.8)
- added D17: YELLOW, LED-3MM-SMD, F.Cu at (89.0, 154.8)
- added D17: YELLOW, LED-3MM-SMD, F.Cu at (84.0, 33.2)
- added D18 (x3): YELLOW, LED-3MM-SMD, F.Cu at (188.0, 28.0)
- added D18 (x2): YELLOW, LED-3MM-SMD, F.Cu at (86.0, 84.0)
- added D18: YELLOW, LED-3MM-SMD, F.Cu at (191.0, 86.0)
- added D18: YELLOW, LED-3MM-SMD, F.Cu at (89.0, 150.0)
- added D18: YELLOW, LED-3MM-SMD, F.Cu at (84.0, 28.5)
- added D2 (x3): GREEN, LED-3MM-SMD, F.Cu at (171.3, 45.4)
- added D2 (x2): GREEN, LED-3MM-SMD, F.Cu at (69.3, 101.4)
- added D2: GREEN, LED-3MM-SMD, F.Cu at (174.3, 103.4)
- added D2: GREEN, LED-3MM-SMD, F.Cu at (72.3, 167.4)
- added D2: GREEN, LED-3MM-SMD, F.Cu at (67.3, 45.9)
- added F1 (x3): FUSE, SM1812, B.Cu at (156.9, 56.8)
- added F1 (x2): FUSE, SM1812, B.Cu at (54.9, 112.8)
- added F1: FUSE, SM1812, B.Cu at (159.9, 114.8)
- added F1: FUSE, SM1812, B.Cu at (57.9, 178.8)
- added F1: FUSE, SM1812, B.Cu at (52.9, 57.3)
- added IC1 (x3): MAX3243, tssop-28, B.Cu at (173.3, 39.5)
- added IC1 (x2): MAX3243, tssop-28, B.Cu at (71.3, 95.5)
- added IC1: MAX3243, tssop-28, B.Cu at (176.3, 97.5)
- added IC1: MAX3243, tssop-28, B.Cu at (74.3, 161.4)
- added IC1: MAX3243, tssop-28, B.Cu at (69.3, 40.0)
- added IC2 (x3): FT232BL, TQFP32, B.Cu at (161.2, 43.0)
- added IC2 (x2): FT232BL, TQFP32, B.Cu at (59.1, 99.0)
- added IC2: FT232BL, TQFP32, B.Cu at (164.2, 101.0)
- added IC2: FT232BL, TQFP32, B.Cu at (62.1, 165.0)
- added IC2: FT232BL, TQFP32, B.Cu at (57.1, 43.5)
- added J1 (x3): COM LEFT, DB9MC-v2, B.Cu at (133.5, 44.5)
- added J1 (x2): COM LEFT, DB9MC-v2, B.Cu at (31.5, 100.5)
- added J1: COM LEFT, DB9MC-v2, B.Cu at (136.5, 102.5)
- added J1: COM LEFT, DB9MC-v2, B.Cu at (34.5, 166.5)
- added J1: COM LEFT, DB9MC-v2, B.Cu at (29.5, 45.0)
- added J2 (x3): COM RIGHT, DB9MC-v2, B.Cu at (204.5, 44.5)
- added J2 (x2): COM RIGHT, DB9MC-v2, B.Cu at (102.5, 100.5)
- added J2: COM RIGHT, DB9MC-v2, B.Cu at (207.5, 102.5)
- added J2: COM RIGHT, DB9MC-v2, B.Cu at (105.5, 166.5)
- added J2: COM RIGHT, DB9MC-v2, B.Cu at (100.5, 45.0)
- added J3 (x3): FTDI, SIL-8, F.Cu at (197.5, 44.5)
- added J3 (x2): FTDI, SIL-8, F.Cu at (95.5, 100.5)
- added J3: FTDI, SIL-8, F.Cu at (200.5, 102.5)
- added J3: FTDI, SIL-8, F.Cu at (98.5, 166.5)
- added J3: FTDI, SIL-8, F.Cu at (93.5, 45.0)
- added J4 (x3): COM RIGHT FTDI, SIL-8, F.Cu at (140.8, 44.5)
- added J4 (x2): COM RIGHT FTDI, SIL-8, F.Cu at (38.8, 100.5)
- added J4: COM RIGHT FTDI, SIL-8, F.Cu at (143.8, 102.5)
- added J4: COM RIGHT FTDI, SIL-8, F.Cu at (41.8, 166.5)
- added J4: COM RIGHT FTDI, SIL-8, F.Cu at (36.8, 45.0)
- added J5 (x3): UART, SIL-4, F.Cu at (168.9, 50.4)
- added J5 (x2): UART, SIL-4, F.Cu at (66.9, 106.4)
- added J5: UART, SIL-4, F.Cu at (171.9, 108.4)
- added J5: UART, SIL-4, F.Cu at (69.9, 172.4)
- added J5: UART, SIL-4, F.Cu at (64.9, 50.9)
- added J6 (x3): COM LEFT COM, SIL-8, F.Cu at (138.2, 44.5)
- added J6 (x2): COM LEFT COM, SIL-8, F.Cu at (36.2, 100.5)
- added J6: COM LEFT COM, SIL-8, F.Cu at (141.2, 102.5)
- added J6: COM LEFT COM, SIL-8, F.Cu at (39.2, 166.5)
- added J6: COM LEFT COM, SIL-8, F.Cu at (34.2, 45.0)
- added J7 (x3): COM RIGHT COM, SIL-8, F.Cu at (200.0, 44.5)
- added J7 (x2): COM RIGHT COM, SIL-8, F.Cu at (98.0, 100.5)
- added J7: COM RIGHT COM, SIL-8, F.Cu at (203.0, 102.5)
- added J7: COM RIGHT COM, SIL-8, F.Cu at (101.0, 166.5)
- added J7: COM RIGHT COM, SIL-8, F.Cu at (96.0, 45.0)
- added L1 (x3): INDUCTOR_SMALL, SM1206, B.Cu at (152.1, 53.8)
- added L1 (x2): INDUCTOR_SMALL, SM1206, B.Cu at (50.1, 109.8)
- added L1: INDUCTOR_SMALL, SM1206, B.Cu at (155.1, 111.8)
- added L1: INDUCTOR_SMALL, SM1206, B.Cu at (53.1, 175.8)
- added L1: INDUCTOR_SMALL, SM1206, B.Cu at (48.1, 54.3)
- added R1 (x3): 470R, SM0805, B.Cu at (155.7, 49.8)
- added R1 (x2): 470R, SM0805, B.Cu at (53.7, 105.8)
- added R1: 470R, SM0805, B.Cu at (158.7, 107.8)
- added R1: 470R, SM0805, B.Cu at (56.7, 171.8)
- added R1: 470R, SM0805, B.Cu at (51.7, 50.3)
- added R10 (x3): 0R, SM0603, B.Cu at (149.1, 60.4)
- added R10 (x2): 0R, SM0603, B.Cu at (47.1, 116.4)
- added R10: 0R, SM0603, B.Cu at (152.1, 118.4)
- added R10: 0R, SM0603, B.Cu at (50.1, 182.4)
- added R10: 0R, SM0603, B.Cu at (45.1, 60.9)
- added R11 (x3): 0R, SM0603, B.Cu at (171.8, 47.4)
- added R11 (x2): 0R, SM0603, B.Cu at (69.8, 103.4)
- added R11: 0R, SM0603, B.Cu at (174.8, 105.4)
- added R11: 0R, SM0603, B.Cu at (72.8, 169.4)
- added R11: 0R, SM0603, B.Cu at (67.8, 47.9)
- added R15 (x3): 470R, SM0805, F.Cu at (178.8, 51.8)
- added R15 (x2): 470R, SM0805, F.Cu at (76.8, 107.8)
- added R15: 470R, SM0805, F.Cu at (181.8, 109.8)
- added R15: 470R, SM0805, F.Cu at (79.8, 173.8)
- added R15: 470R, SM0805, F.Cu at (74.8, 52.2)
- added R16 (x3): 470R, SM0805, F.Cu at (178.8, 49.5)
- added R16 (x2): 470R, SM0805, F.Cu at (76.8, 105.5)
- added R16: 470R, SM0805, F.Cu at (181.8, 107.5)
- added R16: 470R, SM0805, F.Cu at (79.8, 171.5)
- added R16: 470R, SM0805, F.Cu at (74.8, 50.0)
- added R17 (x3): 470R, SM0805, F.Cu at (178.8, 56.2)
- added R17 (x2): 470R, SM0805, F.Cu at (76.8, 112.2)
- added R17: 470R, SM0805, F.Cu at (181.8, 114.2)
- added R17: 470R, SM0805, F.Cu at (79.8, 178.2)
- added R17: 470R, SM0805, F.Cu at (74.8, 56.8)
- added R18 (x3): 470R, SM0805, F.Cu at (178.8, 47.2)
- added R18 (x2): 470R, SM0805, F.Cu at (76.8, 103.2)
- added R18: 470R, SM0805, F.Cu at (181.8, 105.2)
- added R18: 470R, SM0805, F.Cu at (79.8, 169.2)
- added R18: 470R, SM0805, F.Cu at (74.8, 47.8)
- added R19 (x3): 470R, SM0805, F.Cu at (178.8, 54.0)
- added R19 (x2): 470R, SM0805, F.Cu at (76.8, 110.0)
- added R19: 470R, SM0805, F.Cu at (181.8, 112.0)
- added R19: 470R, SM0805, F.Cu at (79.8, 176.0)
- added R19: 470R, SM0805, F.Cu at (74.8, 54.5)
- added R2 (x3): 27R, SM0805, B.Cu at (146.9, 56.2)
- added R2 (x2): 27R, SM0805, B.Cu at (44.9, 112.2)
- added R2: 27R, SM0805, B.Cu at (149.9, 114.2)
- added R2: 27R, SM0805, B.Cu at (47.9, 178.2)
- added R2: 27R, SM0805, B.Cu at (42.9, 56.7)
- added R20 (x3): 470R, SM0805, F.Cu at (178.8, 45.0)
- added R20 (x2): 470R, SM0805, F.Cu at (76.8, 101.0)
- added R20: 470R, SM0805, F.Cu at (181.8, 103.0)
- added R20: 470R, SM0805, F.Cu at (79.8, 167.0)
- added R20: 470R, SM0805, F.Cu at (74.8, 45.5)
- added R21 (x3): 470R, SM0805, F.Cu at (178.8, 42.8)
- added R21 (x2): 470R, SM0805, F.Cu at (76.8, 98.8)
- added R21: 470R, SM0805, F.Cu at (181.8, 100.8)
- added R21: 470R, SM0805, F.Cu at (79.8, 164.8)
- added R21: 470R, SM0805, F.Cu at (74.8, 43.2)
- added R22 (x3): 470R, SM0805, F.Cu at (178.8, 40.5)
- added R22 (x2): 470R, SM0805, F.Cu at (76.8, 96.5)
- added R22: 470R, SM0805, F.Cu at (181.8, 98.5)
- added R22: 470R, SM0805, F.Cu at (79.8, 162.5)
- added R22: 470R, SM0805, F.Cu at (74.8, 41.0)
- added R3 (x3): 27R, SM0805, B.Cu at (149.1, 56.2)
- added R3 (x2): 27R, SM0805, B.Cu at (47.1, 112.2)
- added R3: 27R, SM0805, B.Cu at (152.1, 114.2)
- added R3: 27R, SM0805, B.Cu at (50.1, 178.2)
- added R3: 27R, SM0805, B.Cu at (45.1, 56.7)
- added R4 (x3): 1k5, SM1206, B.Cu at (151.4, 42.8)
- added R4 (x2): 1k5, SM1206, B.Cu at (49.4, 98.8)
- added R4: 1k5, SM1206, B.Cu at (154.4, 100.8)
- added R4: 1k5, SM1206, B.Cu at (52.4, 164.8)
- added R4: 1k5, SM1206, B.Cu at (47.4, 43.2)
- added R5 (x3): R, SM0805, F.Cu at (163.9, 46.7)
- added R5 (x2): R, SM0805, F.Cu at (61.9, 102.7)
- added R5: R, SM0805, F.Cu at (166.9, 104.7)
- added R5: R, SM0805, F.Cu at (64.9, 168.7)
- added R5: R, SM0805, F.Cu at (59.9, 47.2)
- added R6 (x3): R, SM0805, F.Cu at (173.7, 46.7)
- added R6 (x2): R, SM0805, F.Cu at (71.7, 102.7)
- added R6: R, SM0805, F.Cu at (176.7, 104.7)
- added R6: R, SM0805, F.Cu at (74.7, 168.7)
- added R6: R, SM0805, F.Cu at (69.7, 47.2)
- added R7 (x3): 0R, SM0603, B.Cu at (169.3, 45.4)
- added R7 (x2): 0R, SM0603, B.Cu at (67.3, 101.4)
- added R7: 0R, SM0603, B.Cu at (172.3, 103.4)
- added R7: 0R, SM0603, B.Cu at (70.3, 167.4)
- added R7: 0R, SM0603, B.Cu at (65.3, 45.9)
- added R8 (x3): 0R, SM0805, B.Cu at (156.9, 62.4)
- added R8 (x2): 0R, SM0805, B.Cu at (54.9, 118.4)
- added R8: 0R, SM0805, B.Cu at (159.9, 120.4)
- added R8: 0R, SM0805, B.Cu at (57.9, 184.4)
- added R8: 0R, SM0805, B.Cu at (52.9, 62.9)
- added R9 (x3): 0R, SM1206, B.Cu at (163.9, 58.0)
- added R9 (x2): 0R, SM1206, B.Cu at (61.9, 114.0)
- added R9: 0R, SM1206, B.Cu at (166.9, 116.0)
- added R9: 0R, SM1206, B.Cu at (64.9, 180.0)
- added R9: 0R, SM1206, B.Cu at (59.9, 58.5)
- added SIL-1 (x3): Val**, SIL-1, F.Cu at (141.5, 30.5)
- added SIL-1 (x3): Val**, SIL-1, F.Cu at (129.0, 40.5)
- added SIL-1 (x3): Val**, SIL-1, F.Cu at (200.5, 62.5)
- added SIL-1 (x3): Val**, SIL-1, F.Cu at (198.5, 25.0)
- added SIL-1 (x3): Val**, SIL-1, F.Cu at (140.0, 58.5)
- added SIL-1 (x3): Val**, SIL-1, F.Cu at (155.0, 21.5)
- added SIL-1 (x2): Val**, SIL-1, F.Cu at (39.5, 86.5)
- added SIL-1 (x2): Val**, SIL-1, F.Cu at (38.0, 114.5)
- added SIL-1 (x2): Val**, SIL-1, F.Cu at (53.0, 77.5)
- added SIL-1 (x2): Val**, SIL-1, F.Cu at (27.0, 96.5)
- added SIL-1 (x2): Val**, SIL-1, F.Cu at (98.5, 118.5)
- added SIL-1 (x2): Val**, SIL-1, F.Cu at (96.5, 81.0)
- added SIL-1: Val**, SIL-1, F.Cu at (144.5, 88.5)
- added SIL-1: Val**, SIL-1, F.Cu at (143.0, 116.5)
- added SIL-1: Val**, SIL-1, F.Cu at (158.0, 79.5)
- added SIL-1: Val**, SIL-1, F.Cu at (132.0, 98.5)
- added SIL-1: Val**, SIL-1, F.Cu at (203.5, 120.5)
- added SIL-1: Val**, SIL-1, F.Cu at (201.5, 83.0)
- added SIL-1: Val**, SIL-1, F.Cu at (42.5, 152.5)
- added SIL-1: Val**, SIL-1, F.Cu at (41.0, 180.5)
- added SIL-1: Val**, SIL-1, F.Cu at (56.0, 143.5)
- added SIL-1: Val**, SIL-1, F.Cu at (30.0, 162.5)
- added SIL-1: Val**, SIL-1, F.Cu at (101.5, 184.5)
- added SIL-1: Val**, SIL-1, F.Cu at (99.5, 147.0)
- added SIL-1: Val**, SIL-1, F.Cu at (37.5, 31.0)
- added SIL-1: Val**, SIL-1, F.Cu at (36.0, 59.0)
- added SIL-1: Val**, SIL-1, F.Cu at (51.0, 22.0)
- added SIL-1: Val**, SIL-1, F.Cu at (25.0, 41.0)
- added SIL-1: Val**, SIL-1, F.Cu at (96.5, 63.0)
- added SIL-1: Val**, SIL-1, F.Cu at (94.5, 25.5)
Routing:
- net GND: track 0.00 -> 1876.5 mm, vias 0 -> 56
- net /RST COM: track 0.00 -> 922.9 mm
- net /CTS COM: track 0.00 -> 839.5 mm
- net /DSR COM: track 0.00 -> 804.5 mm
- net VCC: track 0.00 -> 799.5 mm, vias 0 -> 16
- net /DTR COM: track 0.00 -> 797.2 mm
- net /RI COM: track 0.00 -> 795.6 mm
- net /RxD COM: track 0.00 -> 776.6 mm
- net /TxD COM: track 0.00 -> 759.7 mm
- net /DCD COM: track 0.00 -> 669.5 mm
- net /D-: track 0.00 -> 304.0 mm
- net /D+: track 0.00 -> 246.0 mm
- net /Tout: RST: track 0.00 -> 209.5 mm
- net /Tout: DTR: track 0.00 -> 203.2 mm
- net /Tout: TxD: track 0.00 -> 196.9 mm
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- added copper zone on B.Cu, net GND
- added copper zone on F.Cu, net GND
Other:
- board size 156.2 x 147.5 mm -> 192 x 173 mm
- net class Default: clearance 0.254 -> 0.2032; trace_width 0.254 -> 0.3556; via_dia 0.889 -> 1.3; via_drill 0.635 -> 0.9
- net class power added: clearance 0.2032, trace_width 0.6096, via_dia 1.3, via_drill 0.9
- net class pwr removed
- net class small track added: clearance 0.2032, trace_width 0.254, via_dia 1.3, via_drill 0.9
- rule trace_clearance: 0.254 -> 0.2032
- rule via_min_drill: 0.508 -> 0.9
- rule via_min_size: 0.889 -> 1.3
