File: led_cube_3x3x3/led_cube_3x3x3_v2.sch (KiCad schematic (older format))
At the start: 66 parts, among them IC1 ATMEGA8A-P, J1 Supply, J2 ISP, J4 UART, P1 CONN_1, P2 CONN_1, P3 CONN_1, P4 CONN_1, P5 CONN_1, P6 CONN_1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

Commit message: led cube sch pcp v2.0
Parts:
- removed P1, P2, P3, P4, P5, P6: CONN_1, symbol CONN_1
- removed R35: 0R, SM0805, symbol R
Connections:
- net labels removed: GNDPWR2
- wire segments 215 -> 210
