File: led_cube_3x3x3/led_cube_3x3x3_v2.kicad_pcb (KiCad board)
At the start: 2 copper layers, 66 x 66 mm, 149 parts, among them IC1 ATMEGA8A-P, J1 Supply, J2 ISP, J4 UART, Q1 A1015, Q2 A1015, Q3 A1015, Q4 SFH320, U1 ST2221C, U2 24C512, X1 16MHz

Commit message: led cube pcb v2.1
Parts:
- removed the ? at (184.2, 94.0)
- removed the ? at (184.0, 89.5)
- removed the ? at (187.8, 88.5)
- removed the ? at (193.0, 83.5)
- removed the ? at (215.2, 83.5)
- removed the ? at (205.0, 83.5)
- removed the ? at (204.5, 86.8)
- removed the ? at (195.8, 86.8)
- removed the ? at (190.8, 91.8)
- removed the ? at (189.0, 81.8)
- removed the ? at (201.0, 80.8)
- removed the ? at (184.2, 101.0)
- removed the ? at (218.0, 81.0)
- removed the ? at (217.5, 83.5)
- removed the ? at (226.5, 83.8)
- removed the ? at (231.2, 82.0)
- removed the ? at (237.8, 88.2)
- removed the ? at (247.0, 90.2)
- removed the ? at (242.5, 96.8)
- removed the ? at (247.0, 100.8)
- removed the ? at (247.2, 114.5)
- removed the ? at (247.2, 129.2)
- removed the ? at (184.5, 116.5)
- removed the ? at (246.0, 143.2)
- removed the ? at (238.0, 144.2)
- removed the ? at (229.8, 143.2)
- removed the ? at (223.0, 137.0)
- removed the ? at (226.2, 133.5)
- removed the ? at (232.5, 132.2)
- removed the ? at (237.5, 132.5)
- removed the ? at (232.8, 140.8)
- removed the ? at (243.0, 140.0)
- removed the ? at (244.5, 132.8)
- removed the ? at (189.5, 121.2)
- removed the ? at (244.8, 122.5)
- removed the ? at (244.5, 105.8)
- removed the ? at (241.2, 112.2)
- removed the ? at (241.0, 119.2)
- removed the ? at (240.2, 126.5)
- removed the ? at (242.0, 136.8)
- removed the ? at (218.8, 140.2)
- removed the ? at (225.5, 129.5)
- removed the ? at (220.8, 123.5)
- removed the ? at (224.2, 119.5)
- removed the ? at (190.0, 132.0)
- removed the ? at (228.2, 121.0)
- removed the ? at (230.2, 117.0)
- removed the ? at (231.5, 112.2)
- removed the ? at (228.5, 109.2)
- removed the ? at (235.2, 102.5)
- removed the ? at (229.0, 104.2)
- removed the ? at (225.5, 100.5)
- removed the ? at (228.0, 89.5)
- removed the ? at (224.2, 89.8)
- removed the ? at (194.8, 128.8)
- removed the ? at (227.5, 86.5)
- removed the ? at (221.0, 86.2)
- removed the ? at (205.2, 91.8)
- removed the ? at (202.8, 96.2)
- removed the ? at (205.8, 100.2)
- removed the ? at (204.5, 116.2)
- removed the ? at (204.2, 120.5)
- removed the ? at (208.8, 127.8)
- removed the ? at (201.2, 128.0)
- removed the ? at (203.0, 136.8)
- removed the ? at (192.8, 117.2)
- removed the ? at (199.8, 144.0)
- removed the ? at (195.2, 139.0)
- removed the ? at (187.5, 142.0)
- removed the ? at (184.8, 126.8)
- removed the ? at (191.5, 93.8)
- removed the ? at (190.5, 105.2)
- removed the ? at (190.5, 98.5)
- removed the ? at (203.2, 109.8)
- removed the ? at (222.0, 109.0)
- removed the ? at (188.2, 108.8)
- removed the ? at (221.5, 102.8)
- removed the ? at (217.8, 99.2)
- removed the ? at (244.2, 82.2)
- removed the ? at (240.8, 93.0)
- removed the ? at (206.0, 114.0)
- removed the ? at (218.5, 116.0)
- removed the ? at (218.0, 119.0)
- removed the ? at (239.5, 108.5)
- removed the ? at (220.5, 128.2)
- removed the ? at (187.5, 93.8)
- removed the ? at (218.5, 112.5)
- added ?: , VIA, F.Cu at (184.5, 128.0)
- added ?: , VIA, F.Cu at (195.5, 129.0)
- added ?: , VIA, F.Cu at (201.0, 129.0)
- added ?: , VIA, F.Cu at (211.4, 130.6)
- added ?: , VIA, F.Cu at (215.2, 138.0)
- added ?: , VIA, F.Cu at (218.5, 141.5)
- added ?: , VIA, F.Cu at (221.2, 137.2)
- added ?: , VIA, F.Cu at (217.2, 132.4)
- added ?: , VIA, F.Cu at (225.6, 129.4)
- added ?: , VIA, F.Cu at (226.0, 133.4)
- added ?: , VIA, F.Cu at (231.8, 133.6)
- added ?: , VIA, F.Cu at (237.8, 132.4)
- added ?: , VIA, F.Cu at (233.0, 141.5)
- added ?: , VIA, F.Cu at (230.5, 144.0)
- added ?: , VIA, F.Cu at (238.4, 144.6)
- added ?: , VIA, F.Cu at (246.4, 143.2)
- added ?: , VIA, F.Cu at (242.5, 141.0)
- added ?: , VIA, F.Cu at (241.8, 137.0)
- added ?: , VIA, F.Cu at (244.5, 134.0)
- added ?: , VIA, F.Cu at (247.2, 130.6)
- added ?: , VIA, F.Cu at (240.0, 127.0)
- added ?: , VIA, F.Cu at (240.2, 119.4)
- added ?: , VIA, F.Cu at (228.2, 120.6)
- added ?: , VIA, F.Cu at (223.4, 119.4)
- added ?: , VIA, F.Cu at (230.2, 117.0)
- added ?: , VIA, F.Cu at (217.8, 119.0)
- added ?: , VIA, F.Cu at (218.2, 116.0)
- added ?: , VIA, F.Cu at (204.8, 123.0)
- added ?: , VIA, F.Cu at (193.4, 118.0)
- added ?: , VIA, F.Cu at (189.5, 122.5)
- added ?: , VIA, F.Cu at (225.2, 138.0)
- added ?: , VIA, F.Cu at (185.0, 117.5)
- added ?: , VIA, F.Cu at (184.0, 87.4)
- added ?: , VIA, F.Cu at (184.2, 95.8)
- added ?: , VIA, F.Cu at (184.2, 107.8)
- added ?: , VIA, F.Cu at (188.0, 107.8)
- added ?: , VIA, F.Cu at (191.2, 106.0)
- added ?: , VIA, F.Cu at (190.4, 99.6)
- added ?: , VIA, F.Cu at (193.2, 93.8)
- added ?: , VIA, F.Cu at (190.6, 91.2)
- added ?: , VIA, F.Cu at (187.4, 99.4)
- added ?: , VIA, F.Cu at (187.4, 140.4)
- added ?: , VIA, F.Cu at (187.8, 88.8)
- added ?: , VIA, F.Cu at (189.0, 81.6)
- added ?: , VIA, F.Cu at (192.4, 84.2)
- added ?: , VIA, F.Cu at (195.4, 87.6)
- added ?: , VIA, F.Cu at (203.8, 86.6)
- added ?: , VIA, F.Cu at (205.0, 83.8)
- added ?: , VIA, F.Cu at (200.8, 80.8)
- added ?: , VIA, F.Cu at (213.2, 83.4)
- added ?: , VIA, F.Cu at (205.0, 91.8)
- added ?: , VIA, F.Cu at (202.4, 95.8)
- added ?: , VIA, F.Cu at (196.0, 140.0)
- added ?: , VIA, F.Cu at (198.0, 101.0)
- added ?: , VIA, F.Cu at (206.2, 101.0)
- added ?: , VIA, F.Cu at (213.6, 111.4)
- added ?: , VIA, F.Cu at (218.4, 112.4)
- added ?: , VIA, F.Cu at (221.8, 108.8)
- added ?: , VIA, F.Cu at (221.6, 103.4)
- added ?: , VIA, F.Cu at (218.0, 100.2)
- added ?: , VIA, F.Cu at (220.2, 83.8)
- added ?: , VIA, F.Cu at (219.6, 81.0)
- added ?: , VIA, F.Cu at (221.0, 86.4)
- added ?: , VIA, F.Cu at (201.0, 144.5)
- added ?: , VIA, F.Cu at (224.0, 89.8)
- added ?: , VIA, F.Cu at (228.4, 89.8)
- added ?: , VIA, F.Cu at (229.8, 94.6)
- added ?: , VIA, F.Cu at (227.4, 86.6)
- added ?: , VIA, F.Cu at (225.6, 83.6)
- added ?: , VIA, F.Cu at (230.4, 81.6)
- added ?: , VIA, F.Cu at (241.0, 82.2)
- added ?: , VIA, F.Cu at (246.4, 89.2)
- added ?: , VIA, F.Cu at (236.4, 88.0)
- added ?: , VIA, F.Cu at (240.4, 93.8)
- added ?: , VIA, F.Cu at (203.5, 137.0)
- added ?: , VIA, F.Cu at (242.8, 97.0)
- added ?: , VIA, F.Cu at (247.0, 101.0)
- added ?: , VIA, F.Cu at (244.8, 107.2)
- added ?: , VIA, F.Cu at (235.2, 102.4)
- added ?: , VIA, F.Cu at (229.6, 105.4)
- added ?: , VIA, F.Cu at (225.8, 101.6)
- added ?: , VIA, F.Cu at (232.2, 105.6)
- added ?: , VIA, F.Cu at (228.4, 110.2)
- added ?: , VIA, F.Cu at (230.6, 112.8)
- added ?: , VIA, F.Cu at (239.0, 109.2)
- added ?: , VIA, F.Cu at (190.5, 133.0)
- added ?: , VIA, F.Cu at (241.0, 112.6)
- added ?: , VIA, F.Cu at (188.2, 113.6)
- added ?: , VIA, F.Cu at (220.6, 123.6)
- added ?: , VIA, F.Cu at (220.0, 128.4)
- added ?: , VIA, F.Cu at (244.8, 124.8)
- added ?: , VIA, F.Cu at (205.6, 117.8)
- added ?: , VIA, F.Cu at (247.4, 115.0)
- added ?: , VIA, F.Cu at (206.0, 113.8)
- added ?: , VIA, F.Cu at (205.6, 109.8)
- moved ? 1.69 mm to (227.4, 93.2)
- moved ? 1.66 mm to (198.2, 98.6)
